Commit message: Add weld seam finding and align the installed camera mount model
Add service-owned bidirectional seam discovery, exposure recovery, native
provenance, measured-section replay and a dedicated JSON-driven Viser panel.
Render the full measured laser profiles and retain portable live scan evidence.
Ship the reproducible Weldfinder seam API patch and independent path auditor.

Align CAD camera and laser centers vertically at the fresh captured rest while
preserving the nominal motion TCP, measured hand-eye and robot dynamics. Add
service-owned read-only disabled rest capture and downward TCP target defaults.
Document the behavior and preserve matching gravity profiles with an XML proof.

Validation: 2095 AutoWeld tests, Ruff, live read-only rest capture, mobile panel
and TCP target checks. Weldfinder validation: 345 tests. Arm remains disabled.

File: assets/camera_mount/camera_mount.urdf (robot description, URDF)
Before this commit: robot yam, 40 links, 39 joints
Links:
- added link weld_tcp
Joints:
- added joint weld_tcp_fixed: type fixed, parent gripper, child weld_tcp, origin xyz=-0.06950000000000001 0.03209562859406243 -0.06878251661400001 rpy=3.141592653589793 0 1.570796326794897
- joint camera_optical_fixed: origin xyz=-0.0695 0.03209562859406243 -0.068782516614 rpy=3.141592653589793 0.0 1.5707963267948966 -> xyz=-0.04176705276517634 0.06349556605564009 -0.06939193296909962 rpy=-3.141592653589793 0.0193916537021086 0.9984603308480584
- joint mount_0_fixed: origin xyz=0.0 0.0 0.0 rpy=0.0 0.0 1.5707963267948966 -> xyz=0 0 0 rpy=5.551115123125783e-17 0.0193916537021086 0.9984603308480582
- joint mount_10_fixed: origin xyz=0.0 0.0 0.0 rpy=0.0 0.0 1.5707963267948966 -> xyz=0 0 0 rpy=5.551115123125783e-17 0.0193916537021086 0.9984603308480582
- joint mount_11_fixed: origin xyz=0.0 0.0 0.0 rpy=0.0 0.0 1.5707963267948966 -> xyz=0 0 0 rpy=5.551115123125783e-17 0.0193916537021086 0.9984603308480582
- joint mount_12_fixed: origin xyz=0.0 0.0 0.0 rpy=0.0 0.0 1.5707963267948966 -> xyz=0 0 0 rpy=5.551115123125783e-17 0.0193916537021086 0.9984603308480582
- joint mount_13_fixed: origin xyz=0.0 0.0 0.0 rpy=0.0 0.0 1.5707963267948966 -> xyz=0 0 0 rpy=5.551115123125783e-17 0.0193916537021086 0.9984603308480582
- joint mount_14_fixed: origin xyz=0.0 0.0 0.0 rpy=0.0 0.0 1.5707963267948966 -> xyz=0 0 0 rpy=5.551115123125783e-17 0.0193916537021086 0.9984603308480582
- joint mount_15_fixed: origin xyz=0.0 0.0 0.0 rpy=0.0 0.0 1.5707963267948966 -> xyz=0 0 0 rpy=5.551115123125783e-17 0.0193916537021086 0.9984603308480582
- joint mount_16_fixed: origin xyz=0.0 0.0 0.0 rpy=0.0 0.0 1.5707963267948966 -> xyz=0 0 0 rpy=5.551115123125783e-17 0.0193916537021086 0.9984603308480582
- joint mount_17_fixed: origin xyz=0.0 0.0 0.0 rpy=0.0 0.0 1.5707963267948966 -> xyz=0 0 0 rpy=5.551115123125783e-17 0.0193916537021086 0.9984603308480582
- joint mount_18_fixed: origin xyz=0.0 0.0 0.0 rpy=0.0 0.0 1.5707963267948966 -> xyz=0 0 0 rpy=5.551115123125783e-17 0.0193916537021086 0.9984603308480582
- joint mount_19_fixed: origin xyz=0.0 0.0 0.0 rpy=0.0 0.0 1.5707963267948966 -> xyz=0 0 0 rpy=5.551115123125783e-17 0.0193916537021086 0.9984603308480582
- joint mount_1_fixed: origin xyz=0.0 0.0 0.0 rpy=0.0 0.0 1.5707963267948966 -> xyz=0 0 0 rpy=5.551115123125783e-17 0.0193916537021086 0.9984603308480582
- joint mount_20_fixed: origin xyz=0.0 0.0 0.0 rpy=0.0 0.0 1.5707963267948966 -> xyz=0 0 0 rpy=5.551115123125783e-17 0.0193916537021086 0.9984603308480582
- joint mount_21_fixed: origin xyz=0.0 0.0 0.0 rpy=0.0 0.0 1.5707963267948966 -> xyz=0 0 0 rpy=5.551115123125783e-17 0.0193916537021086 0.9984603308480582
- joint mount_22_fixed: origin xyz=0.0 0.0 0.0 rpy=0.0 0.0 1.5707963267948966 -> xyz=0 0 0 rpy=5.551115123125783e-17 0.0193916537021086 0.9984603308480582
- joint mount_23_fixed: origin xyz=0.0 0.0 0.0 rpy=0.0 0.0 1.5707963267948966 -> xyz=0 0 0 rpy=5.551115123125783e-17 0.0193916537021086 0.9984603308480582
- joint mount_24_fixed: origin xyz=0.0 0.0 0.0 rpy=0.0 0.0 1.5707963267948966 -> xyz=0 0 0 rpy=5.551115123125783e-17 0.0193916537021086 0.9984603308480582
- joint mount_25_fixed: origin xyz=0.0 0.0 0.0 rpy=0.0 0.0 1.5707963267948966 -> xyz=0 0 0 rpy=5.551115123125783e-17 0.0193916537021086 0.9984603308480582
- joint mount_26_fixed: origin xyz=0.0 0.0 0.0 rpy=0.0 0.0 1.5707963267948966 -> xyz=0 0 0 rpy=5.551115123125783e-17 0.0193916537021086 0.9984603308480582
- joint mount_27_fixed: origin xyz=0.0 0.0 0.0 rpy=0.0 0.0 1.5707963267948966 -> xyz=0 0 0 rpy=5.551115123125783e-17 0.0193916537021086 0.9984603308480582
- joint mount_28_fixed: origin xyz=0.0 0.0 0.0 rpy=0.0 0.0 1.5707963267948966 -> xyz=0 0 0 rpy=5.551115123125783e-17 0.0193916537021086 0.9984603308480582
- joint mount_29_fixed: origin xyz=0.0 0.0 0.0 rpy=0.0 0.0 1.5707963267948966 -> xyz=0 0 0 rpy=5.551115123125783e-17 0.0193916537021086 0.9984603308480582
- joint mount_2_fixed: origin xyz=0.0 0.0 0.0 rpy=0.0 0.0 1.5707963267948966 -> xyz=0 0 0 rpy=5.551115123125783e-17 0.0193916537021086 0.9984603308480582
- joint mount_30_fixed: origin xyz=0.0 0.0 0.0 rpy=0.0 0.0 1.5707963267948966 -> xyz=0 0 0 rpy=5.551115123125783e-17 0.0193916537021086 0.9984603308480582
- joint mount_31_fixed: origin xyz=0.0 0.0 0.0 rpy=0.0 0.0 1.5707963267948966 -> xyz=0 0 0 rpy=5.551115123125783e-17 0.0193916537021086 0.9984603308480582
- joint mount_3_fixed: origin xyz=0.0 0.0 0.0 rpy=0.0 0.0 1.5707963267948966 -> xyz=0 0 0 rpy=5.551115123125783e-17 0.0193916537021086 0.9984603308480582
- joint mount_4_fixed: origin xyz=0.0 0.0 0.0 rpy=0.0 0.0 1.5707963267948966 -> xyz=0 0 0 rpy=5.551115123125783e-17 0.0193916537021086 0.9984603308480582
- joint mount_5_fixed: origin xyz=0.0 0.0 0.0 rpy=0.0 0.0 1.5707963267948966 -> xyz=0 0 0 rpy=5.551115123125783e-17 0.0193916537021086 0.9984603308480582
- joint mount_6_fixed: origin xyz=0.0 0.0 0.0 rpy=0.0 0.0 1.5707963267948966 -> xyz=0 0 0 rpy=5.551115123125783e-17 0.0193916537021086 0.9984603308480582
- joint mount_7_fixed: origin xyz=0.0 0.0 0.0 rpy=0.0 0.0 1.5707963267948966 -> xyz=0 0 0 rpy=5.551115123125783e-17 0.0193916537021086 0.9984603308480582
- joint mount_8_fixed: origin xyz=0.0 0.0 0.0 rpy=0.0 0.0 1.5707963267948966 -> xyz=0 0 0 rpy=5.551115123125783e-17 0.0193916537021086 0.9984603308480582
- joint mount_9_fixed: origin xyz=0.0 0.0 0.0 rpy=0.0 0.0 1.5707963267948966 -> xyz=0 0 0 rpy=5.551115123125783e-17 0.0193916537021086 0.9984603308480582
